File: PCB/Projects/Trigger FPC/FPCJr_Trigger_Board.kicad_sch (KiCad schematic)
At the start: 10 parts, among them J1 Conn_01x05_Pin, J2 Conn_01x05_Pin, U1 HAL4395, U2 HAL4395, U3 HAL4395, U4 HAL4395

Commit message: Flex PCB
Parts:
- removed C3, C4: 100n, Capacitor_SMD:C_0201_0603Metric, symbol Device:C
- removed J1, J2: Conn_01x05_Pin, hhl:505110-0592 Ribbon, symbol Connector:Conn_01x05_Pin
- removed U3, U4: HAL4395, Package_TO_SOT_SMD:SOT-23-5, symbol hhl:HAL4395SO5
- added J1, J2: Conn_01x04_Pin, hhl:505110-0492 Ribbon, symbol Connector:Conn_01x04_Pin
Connections:
- net ADC_2 is gone; now on net ADC_1: U2.5 (OUT)
- net ADC_3 is gone; now on net ADC_0: U1.5 (OUT)
- net +3V3: now also C2.2, U2.1 (IN), J1.1 (Pin_1)
- net +3V3L: now also J2.1 (Pin_1); no longer C2.2, U2.1 (IN)
- net ADC_0: now also J2.3 (Pin_3)
- net ADC_1: now also J1.3 (Pin_3)
- net GND: now also C2.1, U2.2 (GND), J1.4 (Pin_4)
- net GNDL: now also J2.4 (Pin_4); no longer C2.1, U2.2 (GND)
- net TRIGGER_EN_L: now also J2.2 (Pin_2); no longer U2.3 (EN)
- net TRIGGER_EN_R: now also U2.3 (EN), J1.2 (Pin_2)

Commit message: FPC fixes
Parts:
- removed U1, U2: HAL4395, Package_TO_SOT_SMD:SOT-23-5, symbol hhl:HAL4395SO5
- added U1, U2: HAL4395, hhl:SOT-23-5L, symbol Regulator_Linear:TLV70012_SOT23-5
Connections:
- net +3V3: now also U2.1 (VCC)
- net +3V3L: now also U1.1 (VCC)
- net ADC_0: now also U1.5 (OUT)
- net ADC_1: now also U2.5 (OUT)
- net GND: now also U2.3 (GND)
- net GNDL: now also U1.3 (GND)
- net TRIGGER_EN_L: now also U1.2 (~{EN})
- net TRIGGER_EN_R: now also U2.2 (~{EN})
Changed lines of the file:
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@@
 	)
 	(symbol
-		(lib_id "hhl:HAL4395SO5")
-		(at 74.93 58.42 0)
+		(lib_id "Regulator_Linear:TLV70012_SOT23-5")
+		(at 35.56 58.42 0)
 		(unit 1)
 		(exclude_from_sim no)
@@
 		(dnp no)
 		(fields_autoplaced yes)
-		(property "Reference" "U2"
-			(at 74.93 49.53 0)
+		(property "Reference" "U1"
+			(at 35.56 50.8 0)
 			(effects
 				(font
@@
 		)
 		(property "Value" "HAL4395"
-			(at 74.93 52.07 0)
-			(effects
-				(font
-					(size 1.27 1.27)
-				)
-			)
-		)
-		(property "Footprint" "Package_TO_SOT_SMD:SOT-23-5"
-			(at 74.93 50.165 0)
+			(at 35.56 52.832 0)
+			(effects
+				(font
+					(size 1.27 1.27)
+				)
+			)
+		)
+		(property "Footprint" "hhl:SOT-23-5L"
+			(at 35.56 50.165 0)
 			(effects
 				(font
@@
 		)
 		(property "Datasheet" "https://www.lcsc.com/datasheet/C49165022.pdf"
-			(at 74.93 57.15 0)
+			(at 35.814 51.562 0)
 			(effects
 				(font
@@
 		)
 		(property "Description" "SOT-23-5L Linear, Compass (ICs) ROHS"
-			(at 74.93 58.42 0)
-			(effects
-				(font
-					(size 1.27 1.27)
-				)
-				(hide yes)
-			)
-		)
-		(property "Confirmed" ""
-			(at 74.93 58.42 0)
-			(effects
-				(font
-					(size 1.27 1.27)
-				)
-				(hide yes)
-			)
-		)
-		(property "JLCPN" ""
-			(at 74.93 58.42 0)
+			(at 38.608 53.34 0)
+			(effects
+				(font
+					(size 1.27 1.27)
+				)
+				(hide yes)
+			)
+		)
+		(property "Height" ""
+			(at 35.56 58.42 0)
 			(effects
 				(font
@@
 		)
 		(property "LCSC" "C49165022"
-			(at 74.93 58.42 0)
-			(effects
-				(font
-					(size 1.27 1.27)
-				)
-				(hide yes)
-			)
-		)
-		(property "Link" ""
-			(at 74.93 58.42 0)
+			(at 35.56 58.42 0)
 			(effects
 				(font
@@
 		)
 		(property "MPN" "HAL4395SO5"
-			(at 74.93 58.42 0)
+			(at 35.56 58.42 0)
 			(effects
 				(font
@@
 		)
 		(property "Manufacturer" "Hallwee"
-			(at 74.93 58.42 0)
-			(effects
-				(font
-					(size 1.27 1.27)
-				)
-				(hide yes)
-			)
-		)
-		(property "Package" ""
-			(at 74.93 58.42 0)
-			(effects
-				(font
-					(size 1.27 1.27)
-				)
-				(hide yes)
-			)
-		)
-		(property "Price" ""
-			(at 74.93 58.42 0)
-			(effects
-				(font
-					(size 1.27 1.27)
-				)
-				(hide yes)
-			)
+			(at 35.56 58.42 0)
+			(effects
+				(font
+					(size 1.27 1.27)
+				)
+				(hide yes)
+			)
+		)
+		(property "Manufacturer_Name" ""
+			(at 35.56 58.42 0)
+			(effects
+				(font
+					(size 1.27 1.27)
+				)
+				(hide yes)
+			)
+		)
+		(property "Mouser Part Number" ""
+			(at 35.56 58.42 0)
+			(effects
+				(font
+					(size 1.27 1.27)
+				)
+				(hide yes)
+			)
+		)
+		(property "Mouser Price/Stock" ""
+			(at 35.56 58.42 0)
+			(effects
+				(font
+					(size 1.27 1.27)
+				)
+				(hide yes)
+			)
+		)
+		(pin "2"
+		)
+		(pin "5"
+		)
+		(pin "1"
 		)
 		(pin "3"
 		)
-		(pin "5"
-		)
-		(pin "1"
-		)
 		(pin "4"
 		)
-		(pin "2"
-		)
-		(instances
-			(project "FPC_Trigger_Board"
-				(path "/0ea62352-365c-4f6f-aa9e-f2b7bb50112a"
-					(reference "U2")
+		(instances
+			(project "FPCJr_Trigger_Board"
+				(path "/0ea62352-365c-4f6f-aa9e-f2b7bb50112a"
+					(reference "U1")
 					(unit 1)
 				)
@@
 	)
 	(symbol
-		(lib_id "hhl:HAL4395SO5")
-		(at 35.56 58.42 0)
+		(lib_id "Regulator_Linear:TLV70012_SOT23-5")
+		(at 74.93 58.42 0)
 		(unit 1)
 		(exclude_from_sim no)
@@
 		(dnp no)
 		(fields_autoplaced yes)
-		(property "Reference" "U1"
-			(at 35.56 49.53 0)
+		(property "Reference" "U2"
+			(at 74.93 50.8 0)
 			(effects
 				(font
@@
 		)
 		(property "Value" "HAL4395"
-			(at 35.56 52.07 0)
-			(effects
-				(font
-					(size 1.27 1.27)
-				)
-			)
-		)
-		(property "Footprint" "Package_TO_SOT_SMD:SOT-23-5"
-			(at 35.56 50.165 0)
+			(at 74.93 52.832 0)
+			(effects
+				(font
+					(size 1.27 1.27)
+				)
+			)
+		)
+		(property "Footprint" "hhl:SOT-23-5L"
+			(at 74.93 50.165 0)
 			(effects
 				(font
@@
 		)
 		(property "Datasheet" "https://www.lcsc.com/datasheet/C49165022.pdf"
-			(at 35.56 57.15 0)
+			(at 75.184 51.562 0)
 			(effects
 				(font
@@
 		)
 		(property "Description" "SOT-23-5L Linear, Compass (ICs) ROHS"
-			(at 35.56 58.42 0)
-			(effects
-				(font
-					(size 1.27 1.27)
-				)
-				(hide yes)
-			)
-		)
-		(property "Confirmed" ""
-			(at 35.56 58.42 0)
-			(effects
-				(font
-					(size 1.27 1.27)
-				)
-				(hide yes)
-			)
-		)
-		(property "JLCPN" ""
-			(at 35.56 58.42 0)
+			(at 77.978 53.34 0)
+			(effects
+				(font
+					(size 1.27 1.27)
+				)
+				(hide yes)
+			)
+		)
+		(property "Height" ""
+			(at 74.93 58.42 0)
 			(effects
 				(font
@@
 		)
 		(property "LCSC" "C49165022"
-			(at 35.56 58.42 0)
-			(effects
-				(font
-					(size 1.27 1.27)
-				)
-				(hide yes)
-			)
-		)
-		(property "Link" ""
-			(at 35.56 58.42 0)
+			(at 74.93 58.42 0)
 			(effects
 				(font
@@
 		)
 		(property "MPN" "HAL4395SO5"
-			(at 35.56 58.42 0)
+			(at 74.93 58.42 0)
 			(effects
 				(font
@@
 		)
 		(property "Manufacturer" "Hallwee"
-			(at 35.56 58.42 0)
-			(effects
-				(font
-					(size 1.27 1.27)
-				)
-				(hide yes)
-			)
-		)
-		(property "Package" ""
-			(at 35.56 58.42 0)
-			(effects
-				(font
-					(size 1.27 1.27)
-				)
-				(hide yes)
-			)
-		)
-		(property "Price" ""
-			(at 35.56 58.42 0)
-			(effects
-				(font
-					(size 1.27 1.27)
-				)
-				(hide yes)
-			)
+			(at 74.93 58.42 0)
+			(effects
+				(font
+					(size 1.27 1.27)
+				)
+				(hide yes)
+			)
+		)
+		(property "Manufacturer_Name" ""
+			(at 74.93 58.42 0)
+			(effects
+				(font
+					(size 1.27 1.27)
+				)
+				(hide yes)
+			)
+		)
+		(property "Mouser Part Number" ""
+			(at 74.93 58.42 0)
+			(effects
+				(font
+					(size 1.27 1.27)
+				)
+				(hide yes)
+			)
+		)
+		(property "Mouser Price/Stock" ""
+			(at 74.93 58.42 0)
+			(effects
+				(font
+					(size 1.27 1.27)
+				)
+				(hide yes)
+			)
+		)
+		(pin "2"
+		)
+		(pin "5"
+		)
+		(pin "1"
 		)
 		(pin "3"
 		)
-		(pin "5"
-		)
-		(pin "1"
-		)
 		(pin "4"
 		)
-		(pin "2"
-		)
-		(instances
-			(project ""
-				(path "/0ea62352-365c-4f6f-aa9e-f2b7bb50112a"
-					(reference "U1")
-					(unit 1)
-				)
+		(instances
+			(project "FPCJr_Trigger_Board"
+				(path "/0ea62352-365c-4f6f-aa9e-f2b7bb50112a"
+					(reference "U2")
+					(unit 1)
+				)
